File: WindPCB/WindPCB.kicad_sch (KiCad schematic)
At the start: 32 parts, among them J6 Conn_01x04, U2 TSR_1-2450, U3 SeeeduinoXIAO, U4 MCP2562-E-P, U5 TSR1-2433E, U6 LM7806_TO220

Commit message: Work in progress: use a MCP3202 instead of the the ESP32 ADC
Parts:
- removed C6: 330nF, Capacitor_THT:C_Disc_D6.0mm_W2.5mm_P5.00mm, symbol Device:C
- removed U2: TSR_1-2450, Converter_DCDC:Converter_DCDC_TRACO_TSR-1_THT, symbol Regulator_Switching:TSR_1-2450
- removed U6: LM7806_TO220, Package_TO_SOT_THT:TO-220-3_Vertical, symbol Regulator_Linear:LM7806_TO220
- added C3: 100nF, Capacitor_THT:C_Disc_D6.0mm_W2.5mm_P5.00mm, symbol Device:C
- added C6: 330uF, Capacitor_THT:CP_Radial_D6.3mm_P2.50mm, symbol Device:C_Polarized
- added C8: 47nF, Capacitor_THT:C_Disc_D6.0mm_W2.5mm_P5.00mm, symbol Device:C
- added R1: 4K7, Resistor_THT:R_Axial_DIN0204_L3.6mm_D1.6mm_P7.62mm_Horizontal, symbol Device:R
- added U1: 74AHC1G14, Package_TO_SOT_SMD:SOT-23-5_HandSoldering, symbol 74xGxx:74AHC1G14
- added U2: LM7808_TO220, Package_TO_SOT_THT:TO-220-3_Vertical, symbol Regulator_Linear:LM7808_TO220
- added U7: LM7805_TO220, Package_TO_SOT_THT:TO-220-3_Vertical, symbol Regulator_Linear:LM7805_TO220
- C4, C7: value 1nF -> 22nF
- R12: value 3K3 -> 2K2
- R2, R3: value 2K -> 3K3
- R5: value 2K2 -> 4K7
- renumbered RV2 to RV1, RV3 to RV2
Connections:
- net +12V: now also C6.1
- net +3.3V: now also C3.1, U1.3 (GND)
- net +5V: now also C2.1, U7.3 (VO); no longer C2.2, R5.1
- net GND: now also C2.2, C5.2, C3.2, C6.2, C8.2, R1.2, U1.5 (VCC), U2.2 (GND), U7.2 (GND); no longer C2.1, C5.1, R12.2
- net at R4.1: now also U3.11 (PA6_A10_D10_MOSI); no longer U3.4 (PA11_A3_D3)
- net at C7.1, RV1.2: now also U3.3 (PA10_A2_D2); no longer U3.1 (PA02_A0_D0)
- net at AUX1.4 (Pin_4): now also U3.4 (PA11_A3_D3); no longer U3.6 (PA9_A5_D5_SCL)
- net at U4.4 (RXD): now also U3.6 (PA9_A5_D5_SCL); no longer U3.8 (PB09_A7_D7_RX)
- net at JP4.1 (A), U5.1 (Vin): now also U2.1 (VI), U7.1 (VI)
- net at JP3.2 (C), J_VCC1.1: now also R5.2
- net +6V renamed +8V
- net +8V: now also C5.1, U2.3 (VO); no longer C5.2
- new net: U1.4, U3.1 (PA02_A0_D0)
- new net: C8.1, R1.1, R12.1, U1.2
- new net: J_SPEED1.1, R12.2, R5.1
Other:
- note added: "6.2k at 6 V 4.7k at 7 V 3.9k at 8 V"
- moved on the sheet: C1, C2, C5, JP4, R12, R5, U5
